File: Hardware/LD_Breakout/LD_Breakout/LD_Breakout.kicad_pcb (KiCad board)
At the start: 2 copper layers, 26.2 x 18.5 mm, 18 parts

Commit message: Moved breakout boards to separate layouts
Edge cut no work :,(
Parts:
- removed Conn7: LD, MRDT_Connectors:MOLEX_SL_02_Vertical
- removed D8: Green, LED_SMD:LED_0603_1608Metric_Pad1.05x0.95mm_HandSolder
- removed H5, H6, H8, H9: MountingHole, MRDT_Drill_Holes:4_40_Hole_Corner
- removed LD1: D_Laser_Photo_NType, FTIR_Footprints:RLD63NPC5
- removed R13: 300, Resistor_SMD:R_0603_1608Metric_Pad0.98x0.95mm_HandSolder
- removed R14: 85, LED_SMD:LED_0603_1608Metric_Pad1.05x0.95mm_HandSolder
- LD2: moved to B.Cu
- moved H1 77.6 mm to (127.2, 77.3), turned to 90 degrees
- moved H3 67.6 mm to (137.3, 79.8)
- moved LD2 62.1 mm to (132.3, 78.6), turned to 180 degrees
- moved Conn2 56.7 mm to (133.5, 83.8), turned to 180 degrees
- moved D2 54.6 mm to (130.2, 72.2)
- moved R3 50.3 mm to (134.1, 72.2), turned to 180 degrees
- moved R4 49.2 mm to (136.4, 78.6), turned to 180 degrees
- moved H4 48.1 mm to (127.2, 79.9), turned to 180 degrees
- moved H2 36.2 mm to (137.4, 77.3)
Routing:
- net (no net): track 19.9 -> 0.00 mm, vias 1 -> 0
- net +5V: track 0.00 -> 14.2 mm
- net Net-(LD2-Pad2): track 0.00 -> 2.19 mm
- net Net-(D2-A): track 0.00 -> 2.11 mm
- net GND: vias 0 -> 1
- added copper zone on B.Cu, net GND
- added copper zone on F.Cu, net GND
- removed copper zone on B.Cu, net (none)
Other:
- outline, holes or cut-outs redrawn

Commit message: Finishing touches on all boards
Parts:
- added G***: LOGO, LOGO, F.Cu at (128.3, 77.1)
