File: Hardware/LD_Breakout/LD_Breakout.kicad_sch (KiCad schematic)
At the start: 9 parts

Commit message: Fixed footprints
Some resistors still had LED footprints which I had thought I had fixed, but failed because I did not also update the schematic.
Parts:
- R14: footprint LED_SMD:LED_0603_1608Metric_Pad1.05x0.95mm_HandSolder -> Resistor_SMD:R_0603_1608Metric_Pad0.98x0.95mm_HandSolder
Changed lines of the file:
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@@
       (effects (font (size 1.27 1.27)) (justify left))
     )
-    (property "Footprint" "LED_SMD:LED_0603_1608Metric_Pad1.05x0.95mm_HandSolder" (at 96.012 62.865 90)
+    (property "Footprint" "Resistor_SMD:R_0603_1608Metric_Pad0.98x0.95mm_HandSolder" (at 96.012 62.865 90)
       (effects (font (size 1.27 1.27)) hide)
     )
