File: Hardware/FTIR_Main_Hardware/FTIR_Main_Hardware.kicad_pcb (KiCad board)
At the start: 2 copper layers, 85.9 x 53.1 mm, 45 parts, among them J1 RJ45_LED_Shielded, Q1 IRF7606PBF, Q2 BSS138, Q4 IRF7606PBF, Q6 BSS138, U2 D36V28F7, U3 OKI, U4 TMC2208_Breakout, U6 Teensy4.1_DEV-16771

Commit message: Minor Finishing Touches
Parts:
- moved G*** 102.5 mm to (163.5, 83.5)
- moved G*** 92.8 mm to (143.7, 84.0)
- moved G*** 57.9 mm to (117.7, 67.2)
Changed lines of the file:
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@@
     (pad "2" smd rect (at -5.588 0 90) (size 5.08 2.413) (layers "F.Cu" "F.Paste" "F.Mask")
       (net 2 "GND") (pinfunction "Sleve") (pintype "input"))
-    (pad "2" smd rect (at -5.588 0 90) (size 5.08 2.413) (layers "B.Cu" "F.Paste" "F.Mask")
+    (pad "2" smd rect (at -5.588 0 90) (size 5.08 2.413) (layers "B.Cu" "B.Paste" "B.Mask")
       (net 2 "GND") (pinfunction "Sleve") (pintype "input"))
     (pad "2" smd rect (at 5.588 0 90) (size 5.08 2.413) (layers "F.Cu" "F.Paste" "F.Mask")
       (net 2 "GND") (pinfunction "Sleve") (pintype "input"))
-    (pad "2" smd rect (at 5.588 0 90) (size 5.08 2.413) (layers "B.Cu" "F.Paste" "F.Mask")
+    (pad "2" smd rect (at 5.588 0 90) (size 5.08 2.413) (layers "B.Cu" "B.Paste" "B.Mask")
       (net 2 "GND") (pinfunction "Sleve") (pintype "input"))
   )
@@
     (pad "2" smd rect (at -5.588 0) (size 5.08 2.413) (layers "F.Cu" "F.Paste" "F.Mask")
       (net 2 "GND") (pinfunction "Sleve") (pintype "input"))
-    (pad "2" smd rect (at -5.588 0) (size 5.08 2.413) (layers "B.Cu" "F.Paste" "F.Mask")
+    (pad "2" smd rect (at -5.588 0) (size 5.08 2.413) (layers "B.Cu" "B.Paste" "B.Mask")
       (net 2 "GND") (pinfunction "Sleve") (pintype "input"))
     (pad "2" smd rect (at 5.588 0) (size 5.08 2.413) (layers "F.Cu" "F.Paste" "F.Mask")
       (net 2 "GND") (pinfunction "Sleve") (pintype "input"))
-    (pad "2" smd rect (at 5.588 0) (size 5.08 2.413) (layers "B.Cu" "F.Paste" "F.Mask")
+    (pad "2" smd rect (at 5.588 0) (size 5.08 2.413) (layers "B.Cu" "B.Paste" "B.Mask")
       (net 2 "GND") (pinfunction "Sleve") (pintype "input"))
   )
@@
   )
   (footprint "LOGO" (layer "B.Cu")
-    (at 51.556599 73.036351 180)
+    (at 143.656999 84.034551 180)
     (attr board_only exclude_from_pos_files exclude_from_bom)
     (fp_text reference "G***" (at 0 0) (layer "Dwgs.User") hide
@@
   )
   (footprint "LOGO" (layer "B.Cu")
-    (at 60.3504 59.436 180)
+    (at 117.729 67.183 180)
     (attr board_only exclude_from_pos_files exclude_from_bom)
     (fp_text reference "G***" (at 0 0) (layer "Dwgs.User") hide
@@
   )
   (footprint "LOGO" (layer "B.Cu")
-    (at 61.095075 88.845122 180)
+    (at 163.482475 83.460322 180)
     (attr board_only exclude_from_pos_files exclude_from_bom)
     (fp_text reference "G***" (at 0 0) (layer "Dwgs.User") hide

Commit message: Fixed UART
Connections:
- U6 pad 34: UART -> UART_1
- U6 pad 35: UART -> UART_2
Routing:
- net UART: track 45.1 -> 0.00 mm
- net UART_2: track 0.00 -> 22.6 mm
- net UART_1: track 0.00 -> 22.6 mm
Changed lines of the file:
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@@
   (net 63 "unconnected-(U6-RX7-Pad28)")
   (net 64 "unconnected-(U6-A15-Pad39)")
-  (net 65 "UART")
+  (net 65 "UART_1")
   (net 66 "CLK")
   (net 67 "Net-(U6-A17)")
@@
   (net 69 "unconnected-(U6-A1-Pad15)")
   (net 70 "unconnected-(U6-A2-Pad16)")
+  (net 71 "UART_2")
   (footprint "MRDT_Connectors:MOLEX_SL_02_Vertical" (layer "F.Cu")
     (at 130.2385 63.373)
@@
     (pad "MS2" thru_hole circle (at -5.85 3.81 90) (size 1.524 1.524) (drill 1.016) (layers "*.Cu" "*.Mask")
       (net 33 "MS2_CTRL") (pinfunction "MS2") (pintype "input") (solder_mask_margin 0.102))
-    (pad "PDN_UART" thru_hole circle (at -5.85 -1.27 90) (size 1.524 1.524) (drill 1.016) (layers "*.Cu" "*.Mask")
-      (net 65 "UART") (pinfunction "PDN_UART") (pintype "input") (solder_mask_margin 0.102))
-    (pad "PDN_UART" thru_hole circle (at -5.85 1.27 90) (size 1.524 1.524) (drill 1.016) (layers "*.Cu" "*.Mask")
-      (net 65 "UART") (pinfunction "PDN_UART") (pintype "input") (solder_mask_margin 0.102))
+    (pad "PDN_UART_1" thru_hole circle (at -5.85 1.27 90) (size 1.524 1.524) (drill 1.016) (layers "*.Cu" "*.Mask")
+      (net 65 "UART_1") (pinfunction "PDN_UART_1") (pintype "input") (solder_mask_margin 0.102))
+    (pad "PDN_UART_2" thru_hole circle (at -5.85 -1.27 90) (size 1.524 1.524) (drill 1.016) (layers "*.Cu" "*.Mask")
+      (net 71 "UART_2") (pinfunction "PDN_UART_2") (pintype "input") (solder_mask_margin 0.102))
     (pad "STEP" thru_hole circle (at -5.85 -6.35 90) (size 1.524 1.524) (drill 1.016) (layers "*.Cu" "*.Mask")
       (net 46 "STEP") (pinfunction "STEP") (pintype "input") (solder_mask_margin 0.102))
@@
       (net 44 "BUCK_EN") (pinfunction "MCLK2") (pintype "bidirectional"))
     (pad "34" thru_hole circle (at 26.67 -7.62) (size 1.308 1.308) (drill 0.8) (layers "*.Cu" "*.Mask")
-      (net 65 "UART") (pinfunction "RX8") (pintype "bidirectional"))
+      (net 65 "UART_1") (pinfunction "RX8") (pintype "bidirectional"))
     (pad "35" thru_hole circle (at 24.13 -7.62) (size 1.308 1.308) (drill 0.8) (layers "*.Cu" "*.Mask")
-      (net 65 "UART") (pinfunction "TX8") (pintype "bidirectional"))
+      (net 71 "UART_2") (pinfunction "TX8") (pintype "bidirectional"))
     (pad "36" thru_hole circle (at 21.59 -7.62) (size 1.308 1.308) (drill 0.8) (layers "*.Cu" "*.Mask")
       (net 66 "CLK") (pinfunction "CS2") (pintype "bidirectional"))
@@
   (segment (start 167.8432 102.8192) (end 114.6556 102.8192) (width 0.254) (layer "B.Cu") (net 51))
   (segment (start 114.6556 102.8192) (end 110.744 98.9076) (width 0.254) (layer "B.Cu") (net 51))
-  (segment (start 171.647851 85.8012) (end 167.1828 85.8012) (width 0.254) (layer "F.Cu") (net 65))
-  (segment (start 176.4792 81.6944) (end 172.384887 85.788713) (width 0.254) (layer "F.Cu") (net 65))
-  (segment (start 159.890857 92.3876) (end 166.985257 85.2932) (width 0.254) (layer "F.Cu") (net 65))
-  (segment (start 172.384887 85.788713) (end 171.660338 85.788713) (width 0.254) (layer "F.Cu") (net 65))
-  (segment (start 166.985257 85.2932) (end 170.3404 85.2932) (width 0.254) (layer "F.Cu") (net 65))
-  (segment (start 156.464 93.98) (end 158.0564 92.3876) (width 0.254) (layer "F.Cu") (net 65))
-  (segment (start 170.3404 85.2932) (end 173.9392 81.6944) (width 0.254) (layer "F.Cu") (net 65))
-  (segment (start 158.0564 92.3876) (end 159.890857 92.3876) (width 0.254) (layer "F.Cu") (net 65))
-  (segment (start 171.660338 85.788713) (end 171.647851 85.8012) (width 0.254) (layer "F.Cu") (net 65))
-  (segment (start 167.1828 85.8012) (end 159.004 93.98) (width 0.254) (layer "F.Cu") (net 65))
+  (segment (start 172.4264 85.7472) (end 176.4792 81.6944) (width 0.254) (layer "F.Cu") (net 65))
+  (segment (start 167.2368 85.7472) (end 172.4264 85.7472) (width 0.254) (layer "F.Cu") (net 65))
+  (segment (start 167.2368 85.7472) (end 159.004 93.98) (width 0.254) (layer "F.Cu") (net 65))
   (segment (start 171.3992 81.6944) (end 168.2544 84.8392) (width 0.254) (layer "F.Cu") (net 66))
   (segment (start 168.2544 84.8392) (end 166.797204 84.8392) (width 0.254) (layer "F.Cu") (net 66))
@@
   (segment (start 160.1724 64.6176) (end 161.4932 63.2968) (width 0.254) (layer "F.Cu") (net 68))
   (segment (start 160.1724 68.9318) (end 160.1686 68.9356) (width 0.254) (layer "F.Cu") (net 68))
+  (segment (start 170.3404 85.2932) (end 173.9392 81.6944) (width 0.254) (layer "F.Cu") (net 71))
+  (segment (start 159.890857 92.3876) (end 166.985257 85.2932) (width 0.254) (layer "F.Cu") (net 71))
+  (segment (start 166.985257 85.2932) (end 170.3404 85.2932) (width 0.254) (layer "F.Cu") (net 71))
+  (segment (start 156.464 93.98) (end 158.0564 92.3876) (width 0.254) (layer "F.Cu") (net 71))
+  (segment (start 158.0564 92.3876) (end 159.890857 92.3876) (width 0.254) (layer "F.Cu") (net 71))
   (zone (net 2) (net_name "GND") (layers "F&B.Cu") (hatch edge 0.5)
     (priority 2)

Commit message: Changed UART circuit
Added a resistor to match this diagram:
https://wiki.fysetc.com/TMC2208/#hardware-connection
Parts:
- added R5: 1k, Resistor_SMD:R_0603_1608Metric_Pad0.98x0.95mm_HandSolder, F.Cu at (172.9, 84.2)
- U4: value TMC2208_Breakout -> TMC2208
Connections:
- U4 pad PDN_UART_1: UART_1 -> UART
- U4 pad PDN_UART_2: UART_2 -> UART
- U6 pad 34: UART_1 -> UART
- U6 pad 35: UART_2 -> Net-(U6-TX8)
Routing:
- net UART: track 0.00 -> 25.2 mm
- net UART_2: track 22.6 -> 0.00 mm
- net UART_1: track 22.6 -> 0.00 mm
- net Net-(U6-TX8): track 0.00 -> 19.5 mm
Changed lines of the file:
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@@
   (net 63 "unconnected-(U6-RX7-Pad28)")
   (net 64 "unconnected-(U6-A15-Pad39)")
-  (net 65 "UART_1")
+  (net 65 "UART")
   (net 66 "CLK")
   (net 67 "Net-(U6-A17)")
@@
   (net 69 "unconnected-(U6-A1-Pad15)")
   (net 70 "unconnected-(U6-A2-Pad16)")
-  (net 71 "UART_2")
+  (net 71 "Net-(U6-TX8)")
   (footprint "MRDT_Connectors:MOLEX_SL_02_Vertical" (layer "F.Cu")
     (at 130.2385 63.373)
@@
         (effects (font (size 1.4 1.4) (thickness 0.15)))
     )
-    (fp_text value "TMC2208_Breakout" (at -8.6106 0) (layer "F.SilkS")
+    (fp_text value "TMC2208" (at -8.5344 4.826) (layer "F.SilkS")
         (effects (font (size 1.4 1.4) (thickness 0.15)))
     )
@@
       (net 33 "MS2_CTRL") (pinfunction "MS2") (pintype "input") (solder_mask_margin 0.102))
     (pad "PDN_UART_1" thru_hole circle (at -5.85 1.27 90) (size 1.524 1.524) (drill 1.016) (layers "*.Cu" "*.Mask")
-      (net 65 "UART_1") (pinfunction "PDN_UART_1") (pintype "input") (solder_mask_margin 0.102))
+      (net 65 "UART") (pinfunction "PDN_UART_1") (pintype "input") (solder_mask_margin 0.102))
     (pad "PDN_UART_2" thru_hole circle (at -5.85 -1.27 90) (size 1.524 1.524) (drill 1.016) (layers "*.Cu" "*.Mask")
-      (net 71 "UART_2") (pinfunction "PDN_UART_2") (pintype "input") (solder_mask_margin 0.102))
+      (net 65 "UART") (pinfunction "PDN_UART_2") (pintype "input") (solder_mask_margin 0.102))
     (pad "STEP" thru_hole circle (at -5.85 -6.35 90) (size 1.524 1.524) (drill 1.016) (layers "*.Cu" "*.Mask")
       (net 46 "STEP") (pinfunction "STEP") (pintype "input") (solder_mask_margin 0.102))
@@
       (net 44 "BUCK_EN") (pinfunction "MCLK2") (pintype "bidirectional"))
     (pad "34" thru_hole circle (at 26.67 -7.62) (size 1.308 1.308) (drill 0.8) (layers "*.Cu" "*.Mask")
-      (net 65 "UART_1") (pinfunction "RX8") (pintype "bidirectional"))
+      (net 65 "UART") (pinfunction "RX8") (pintype "bidirectional"))
     (pad "35" thru_hole circle (at 24.13 -7.62) (size 1.308 1.308) (drill 0.8) (layers "*.Cu" "*.Mask")
-      (net 71 "UART_2") (pinfunction "TX8") (pintype "bidirectional"))
+      (net 71 "Net-(U6-TX8)") (pinfunction "TX8") (pintype "bidirectional"))
     (pad "36" thru_hole circle (at 21.59 -7.62) (size 1.308 1.308) (drill 0.8) (layers "*.Cu" "*.Mask")
       (net 66 "CLK") (pinfunction "CS2") (pintype "bidirectional"))
@@
       (clearance 2.5))
   )
+  (footprint "Resistor_SMD:R_0603_1608Metric_Pad0.98x0.95mm_HandSolder" (layer "F.Cu")
+    (at 172.8724 84.2264 180)
+    (descr "Resistor SMD 0603 (1608 Metric), square (rectangular) end terminal, IPC_7351 nominal with elongated pad for handsoldering. (Body size source: IPC-SM-782 page 72, https://www.pcb-3d.com/wordpress/wp-content/uploads/ipc-sm-782a_amendment_1_and_2.pdf), generated with kicad-footprint-generator")
+    (tags "resistor handsolder")
+    (property "Sheetfile" "FTIR_Main_Hardware.kicad_sch")
+    (property "Sheetname" "")
+    (property "ki_description" "Resistor")
+    (property "ki_keywords" "R res resistor")
+    (attr smd)
+    (fp_text reference "R5" (at 2.7432 0) (layer "F.SilkS")
+        (effects (font (size 1 1) (thickness 0.15)))
+    )
+    (fp_text value "1k" (at 0 1.43) (layer "F.Fab")
+        (effects (font (size 1 1) (thickness 0.15)))
+    )
+    (fp_text user "${REFERENCE}" (at 0 0) (layer "F.Fab")
+        (effects (font (size 0.4 0.4) (thickness 0.06)))
+    )
+    (fp_line (start -0.254724 -0.5225) (end 0.254724 -0.5225)
+      (stroke (width 0.12) (type solid)) (layer "F.SilkS"))
+    (fp_line (start -0.254724 0.5225) (end 0.254724 0.5225)
+      (stroke (width 0.12) (type solid)) (layer "F.SilkS"))
+    (fp_line (start -1.65 -0.73) (end 1.65 -0.73)
+      (stroke (width 0.05) (type solid)) (layer "F.CrtYd"))
+    (fp_line (start -1.65 0.73) (end -1.65 -0.73)
+      (stroke (width 0.05) (type solid)) (layer "F.CrtYd"))
+    (fp_line (start 1.65 -0.73) (end 1.65 0.73)
+      (stroke (width 0.05) (type solid)) (layer "F.CrtYd"))
+    (fp_line (start 1.65 0.73) (end -1.65 0.73)
+      (stroke (width 0.05) (type solid)) (layer "F.CrtYd"))
+    (fp_line (start -0.8 -0.4125) (end 0.8 -0.4125)
+      (stroke (width 0.1) (type solid)) (layer "F.Fab"))
+    (fp_line (start -0.8 0.4125) (end -0.8 -0.4125)
+      (stroke (width 0.1) (type solid)) (layer "F.Fab"))
+    (fp_line (start 0.8 -0.4125) (end 0.8 0.4125)
+      (stroke (width 0.1) (type solid)) (layer "F.Fab"))
+    (fp_line (start 0.8 0.4125) (end -0.8 0.4125)
+      (stroke (width 0.1) (type solid)) (layer "F.Fab"))
+    (pad "1" smd roundrect (at -0.9125 0 180) (size 0.975 0.95) (layers "F.Cu" "F.Paste" "F.Mask") (roundrect_rratio 0.25)
+      (net 65 "UART") (pintype "passive"))
+    (pad "2" smd roundrect (at 0.9125 0 180) (size 0.975 0.95) (layers "F.Cu" "F.Paste" "F.Mask") (roundrect_rratio 0.25)
+      (net 71 "Net-(U6-TX8)") (pintype "passive"))
+    (model "${KICAD6_3DMODEL_DIR}/Resistor_SMD.3dshapes/R_0603_1608Metric.wrl"
+      (offset (xyz 0 0 0))
+      (scale (xyz 1 1 1))
+      (rotate (xyz 0 0 0))
+    )
+  )
   (footprint "LED_SMD:LED_0603_1608Metric_Pad1.05x0.95mm_HandSolder" (layer "F.Cu")
     (at 135.9014 71.7026 180)
@@
   (segment (start 167.8432 102.8192) (end 114.6556 102.8192) (width 0.254) (layer "B.Cu") (net 51))
   (segment (start 114.6556 102.8192) (end 110.744 98.9076) (width 0.254) (layer "B.Cu") (net 51))
-  (segment (start 172.4264 85.7472) (end 176.4792 81.6944) (width 0.254) (layer "F.Cu") (net 65))
-  (segment (start 167.2368 85.7472) (end 172.4264 85.7472) (width 0.254) (layer "F.Cu") (net 65))
-  (segment (start 167.2368 85.7472) (end 159.004 93.98) (width 0.254) (layer "F.Cu") (net 65))
-  (segment (start 171.3992 81.6944) (end 168.2544 84.8392) (width 0.254) (layer "F.Cu") (net 66))
-  (segment (start 168.2544 84.8392) (end 166.797204 84.8392) (width 0.254) (layer "F.Cu") (net 66))
-  (segment (start 155.9704 91.9336) (end 153.924 93.98) (width 0.254) (layer "F.Cu") (net 66))
-  (segment (start 166.797204 84.8392) (end 159.702804 91.9336) (width 0.254) (layer "F.Cu") (net 66))
+  (segment (start 173.7849 84.2264) (end 173.9472 84.2264) (width 0.254) (layer "F.Cu") (net 65))
+  (segment (start 159.004 93.98) (end 159.004 93.91368) (width 0.25) (layer "F.Cu") (net 65))
+  (segment (start 173.9392 84.0721) (end 173.9392 81.6944) (width 0.254) (layer "F.Cu") (net 65))
+  (segment (start 173.7849 84.2264) (end 173.9392 84.0721) (width 0.254) (layer "F.Cu") (net 65))
+  (segment (start 159.004 93.91368) (end 167.37888 85.5388) (width 0.25) (layer "F.Cu") (net 65))
+  (segment (start 173.9472 84.2264) (end 176.4792 81.6944) (width 0.254) (layer "F.Cu") (net 65))
+  (segment (start 172.4725 85.5388) (end 173.7849 84.2264) (width 0.25) (layer "F.Cu") (net 65))
+  (segment (start 167.37888 85.5388) (end 172.4725 85.5388) (width 0.25) (layer "F.Cu") (net 65))
   (segment (start 159.702804 91.9336) (end 155.9704 91.9336) (width 0.254) (layer "F.Cu") (net 66))
+  (segment (start 155.9704 91.9336) (end 153.924 93.98) (width 0.254) (layer "F.Cu") (net 66))
+  (segment (start 171.3992 81.6944) (end 168.4608 84.6328) (width 0.254) (layer "F.Cu") (net 66))
+  (segment (start 167.003604 84.6328) (end 159.702804 91.9336) (width 0.254) (layer "F.Cu") (net 66))
+  (segment (start 168.4608 84.6328) (end 167.003604 84.6328) (width 0.254) (layer "F.Cu") (net 66))
   (segment (start 152.2476 64.5668) (end 152.2476 68.8848) (width 0.254) (layer "F.Cu") (net 67))
   (segment (start 141.224 91.0336) (end 153.5176 78.74) (width 0.254) (layer "F.Cu") (net 67))
@@
   (segment (start 160.1724 64.6176) (end 161.4932 63.2968) (width 0.254) (layer "F.Cu") (net 68))
   (segment (start 160.1724 68.9318) (end 160.1686 68.9356) (width 0.254) (layer "F.Cu") (net 68))
-  (segment (start 170.3404 85.2932) (end 173.9392 81.6944) (width 0.254) (layer "F.Cu") (net 71))
-  (segment (start 159.890857 92.3876) (end 166.985257 85.2932) (width 0.254) (layer "F.Cu") (net 71))
-  (segment (start 166.985257 85.2932) (end 170.3404 85.2932) (width 0.254) (layer "F.Cu") (net 71))
-  (segment (start 156.464 93.98) (end 158.0564 92.3876) (width 0.254) (layer "F.Cu") (net 71))
+  (segment (start 167.191657 85.0868) (end 171.0995 85.0868) (width 0.254) (layer "F.Cu") (net 71))
   (segment (start 158.0564 92.3876) (end 159.890857 92.3876) (width 0.254) (layer "F.Cu") (net 71))
+  (segment (start 171.0995 85.0868) (end 171.9599 84.2264) (width 0.254) (layer "F.Cu") (net 71))
+  (segment (start 159.890857 92.3876) (end 167.191657 85.0868) (width 0.254) (layer "F.Cu") (net 71))
+  (segment (start 156.464 93.98) (end 158.0564 92.3876) (width 0.254) (layer "F.Cu") (net 71))
   (zone (net 2) (net_name "GND") (layers "F&B.Cu") (hatch edge 0.5)
     (priority 2)

Commit message: Added 3v3 indicator
also tried to make a gerb, but I don't think it looks quite right
Parts:
- added D1: Green, LED_SMD:LED_0603_1608Metric_Pad1.05x0.95mm_HandSolder, F.Cu at (136.8, 79.5)
- added R6: 100, Resistor_SMD:R_0603_1608Metric_Pad0.98x0.95mm_HandSolder, F.Cu at (133.0, 79.5)
- moved R7 1.35 mm to (132.9, 70.6)
- moved D5 1.35 mm to (136.7, 70.6)
- moved D2 1.35 mm to (136.8, 73.6)
- moved D4 1.35 mm to (136.7, 76.6)
- moved R3 1.35 mm to (133.0, 73.6)
- moved R4 1.35 mm to (133.0, 76.6)
Routing:
- net +3V3: track 122.5 -> 132.2 mm
- net +5V: track 89.8 -> 95.5 mm
- net Net-(D1-A): track 0.00 -> 1.97 mm
- net +12V: track 118.4 -> 119.8 mm
- net +7.5V: track 87.8 -> 89.2 mm
- net GND: vias 0 -> 4
Other:
- board text added: "+3.3V"
